File: C264Cart.kicad_sch (KiCad schematic)
At the start: 3 parts, among them U1 27C512, U2 27C512, U3 264-Exp-Port

Commit message: Work in progress.
Connections:
- net A0: now reaches U2.10 (A0)
- net A0: now also U1.10 (A0), U3.Y (A0)
- net D0: now reaches U2.11 (D0)
- net D0: now also U1.11 (D0), U3.21 (D0)
- net D1: now reaches U2.12 (D1)
- net D1: now also U1.12 (D1), U3.20 (D1)
- net D2: now reaches U2.13 (D2)
- net D2: now also U1.13 (D2), U3.19 (D2)
- net GND: now reaches U2.14 (GND)
- net GND: now also U1.14 (GND)
- net D3: now reaches U2.15 (D3)
- net D3: now also U1.15 (D3), U3.18 (D3)
- net D4: now reaches U2.16 (D4)
- net D4: now also U1.16 (D4), U3.17 (D4)
- net D5: now reaches U2.17 (D5)
- net D5: now also U1.17 (D5), U3.16 (D5)
- net D6: now reaches U2.18 (D6)
- net D6: now also U1.18 (D6), U3.15 (D6)
- net D7: now reaches U2.19 (D7)
- net D7: now also U1.19 (D7), U3.14 (D7)
- net A10: now reaches U2.21 (A10)
- net A10: now also U1.21 (A10), U3.M (A10)
- net A9: now reaches U2.24 (A9)
- net A9: now also U1.24 (A9), U3.N (A9)
- net A8: now reaches U2.25 (A8)
- net A8: now also U1.25 (A8), U3.P (A8)
- net +5V: now reaches U2.28 (VCC)
- net +5V: now also U1.28 (VCC)
- net A7: now reaches U2.3 (A7)
- net A7: now also U1.3 (A7), U3.R (A7)
- net A6: now reaches U2.4 (A6)
- net A6: now also U1.4 (A6), U3.S (A6)
- net A5: now reaches U2.5 (A5)
- net A5: now also U1.5 (A5), U3.T (A5)
- net A4: now reaches U2.6 (A4)
- net A4: now also U1.6 (A4), U3.U (A4)
- net A3: now reaches U2.7 (A3)
- net A3: now also U1.7 (A3), U3.V (A3)
- net A2: now reaches U2.8 (A2)
- net A2: now also U1.8 (A2), U3.W (A2)
- net A1: now reaches U2.9 (A1)
- net A1: now also U1.9 (A1), U3.X (A1)
- no-connect marks 0 -> 3
Other:
- moved on the sheet: U1, U2, U3

Commit message: Work in progress.
Connections:
- net +5V: now also U3.2 (+5V), U3.3 (+5V)
- net GND: now also U3.1 (GND), U3.25 (GND), U3.A (GND), U3.CC (GND)
Changed lines of the file:
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@@
   (junction (at 170.18 54.61) (diameter 0) (color 0 0 0 0)
   )
+  (junction (at 60.96 78.74) (diameter 0) (color 0 0 0 0)
+  )
   (junction (at 137.16 62.23) (diameter 0) (color 0 0 0 0)
+  )
+  (junction (at 113.03 137.16) (diameter 0) (color 0 0 0 0)
+  )
+  (junction (at 113.03 144.78) (diameter 0) (color 0 0 0 0)
+  )
+  (junction (at 113.03 76.2) (diameter 0) (color 0 0 0 0)
   )
   (no_connect (at 101.6 132.08))
@@
     (stroke (width 0) (type default))
   )
+  (wire (pts (xy 60.96 78.74) (xy 60.96 81.28))
+    (stroke (width 0) (type default))
+  )
   (wire (pts (xy 186.69 99.06) (xy 190.5 99.06))
     (stroke (width 0) (type default))
@@
     (stroke (width 0) (type default))
   )
+  (wire (pts (xy 63.5 64.77) (xy 113.03 64.77))
+    (stroke (width 0) (type default))
+  )
   (bus (pts (xy 170.18 54.61) (xy 170.18 78.74))
     (stroke (width 0) (type default))
@@
     (stroke (width 0) (type default))
   )
+  (wire (pts (xy 113.03 137.16) (xy 113.03 144.78))
+    (stroke (width 0) (type default))
+  )
   (wire (pts (xy 163.83 91.44) (xy 167.64 91.44))
     (stroke (width 0) (type default))
@@
     (stroke (width 0) (type default))
   )
+  (wire (pts (xy 60.96 81.28) (xy 63.5 81.28))
+    (stroke (width 0) (type default))
+  )
   (bus (pts (xy 170.18 86.36) (xy 170.18 88.9))
     (stroke (width 0) (type default))
@@
     (stroke (width 0) (type default))
   )
+  (wire (pts (xy 60.96 78.74) (xy 63.5 78.74))
+    (stroke (width 0) (type default))
+  )
   (bus (pts (xy 107.95 121.92) (xy 107.95 119.38))
     (stroke (width 0) (type default))
@@
     (stroke (width 0) (type default))
   )
+  (wire (pts (xy 60.96 137.16) (xy 60.96 144.78))
+    (stroke (width 0) (type default))
+  )
   (bus (pts (xy 184.15 78.74) (xy 184.15 81.28))
     (stroke (width 0) (type default))
@@
     (stroke (width 0) (type default))
   )
+  (wire (pts (xy 101.6 137.16) (xy 113.03 137.16))
+    (stroke (width 0) (type default))
+  )
   (bus (pts (xy 137.16 88.9) (xy 137.16 91.44))
     (stroke (width 0) (type default))
@@
     (stroke (width 0) (type default))
   )
+  (wire (pts (xy 60.96 63.5) (xy 60.96 78.74))
+    (stroke (width 0) (type default))
+  )
   (wire (pts (xy 139.7 76.2) (xy 143.51 76.2))
     (stroke (width 0) (type default))
@@
     (stroke (width 0) (type default))
   )
+  (wire (pts (xy 63.5 137.16) (xy 60.96 137.16))
+    (stroke (width 0) (type default))
+  )
   (wire (pts (xy 59.69 106.68) (xy 63.5 106.68))
     (stroke (width 0) (type default))
@@
     (stroke (width 0) (type default))
   )
+  (wire (pts (xy 113.03 144.78) (xy 113.03 147.32))
+    (stroke (width 0) (type default))
+  )
   (bus (pts (xy 217.17 78.74) (xy 217.17 81.28))
     (stroke (width 0) (type default))
@@
     (stroke (width 0) (type default))
   )
+  (wire (pts (xy 113.03 137.16) (xy 113.03 76.2))
+    (stroke (width 0) (type default))
+  )
   (wire (pts (xy 163.83 86.36) (xy 167.64 86.36))
     (stroke (width 0) (type default))
@@
     (stroke (width 0) (type default))
   )
+  (wire (pts (xy 113.03 76.2) (xy 101.6 76.2))
+    (stroke (width 0) (type default))
+  )
   (wire (pts (xy 59.69 109.22) (xy 63.5 109.22))
     (stroke (width 0) (type default))
@@
     (stroke (width 0) (type default))
   )
+  (wire (pts (xy 60.96 144.78) (xy 113.03 144.78))
+    (stroke (width 0) (type default))
+  )
   (wire (pts (xy 186.69 81.28) (xy 190.5 81.28))
     (stroke (width 0) (type default))
@@
     (stroke (width 0) (type default))
   )
+  (wire (pts (xy 63.5 64.77) (xy 63.5 76.2))
+    (stroke (width 0) (type default))
+  )
   (wire (pts (xy 139.7 91.44) (xy 143.51 91.44))
+    (stroke (width 0) (type default))
+  )
+  (wire (pts (xy 113.03 64.77) (xy 113.03 76.2))
     (stroke (width 0) (type default))
   )
@@
         (path "/7006651b-1f52-4ff6-87a6-d875cc82c860"
           (reference "#PWR06") (unit 1)
+        )
+      )
+    )
+  )
+  (symbol (lib_id "power:GND") (at 113.03 147.32 0) (unit 1)
+    (in_bom yes) (on_board yes) (dnp no) (fields_autoplaced)
+    (property "Reference" "#PWR07" (at 113.03 153.67 0)
+      (effects (font (size 1.27 1.27)) hide)
+    )
+    (property "Value" "GND" (at 113.03 151.4531 0)
+      (effects (font (size 1.27 1.27)))
+    )
+    (property "Footprint" "" (at 113.03 147.32 0)
+      (effects (font (size 1.27 1.27)) hide)
+    )
+    (property "Datasheet" "" (at 113.03 147.32 0)
+      (effects (font (size 1.27 1.27)) hide)
+    )
+    (pin "1")
+    (instances
+      (project "C264Cart"
+        (path "/7006651b-1f52-4ff6-87a6-d875cc82c860"
+          (reference "#PWR07") (unit 1)
         )
       )
@@
         )
       )
+    )
+  )
+  (symbol (lib_id "power:+5V") (at 60.96 63.5 0) (unit 1)
+    (in_bom yes) (on_board yes) (dnp no) (fields_autoplaced)
+    (property "Reference" "#PWR08" (at 60.96 67.31 0)
+      (effects (font (size 1.27 1.27)) hide)
+    )
+    (property "Value" "+5V" (at 60.96 59.3669 0)
+      (effects (font (size 1.27 1.27)))
+    )
+    (property "Footprint" "" (at 60.96 63.5 0)
+      (effects (font (size 1.27 1.27)) hide)
+    )
+    (property "Datasheet" "" (at 60.96 63.5 0)
+      (effects (font (size 1.27 1.27)) hide)
+    )
+    (pin "1")
+    (instances
+      (project "C264Cart"
+        (path "/7006651b-1f52-4ff6-87a6-d875cc82c860"
+          (reference "#PWR08") (unit 1)
+        )
+      )

Commit message: Work in progress.
Parts:
- added J1, J4: SJ, C264Cart:SolderJumper-3_Bridged12-wide, symbol Jumper:SolderJumper_3_Bridged12
- added J2, J5: SJ, C264Cart:SolderJumper-3_Bridged12, symbol Jumper:SolderJumper_3_Bridged12
- added J3, J6: SJ, C264Cart:SolderJumper-3_Bridged12-narrow, symbol Jumper:SolderJumper_3_Bridged12
- added U4: 23128, symbol hackup:23128
Connections:
- net +5V: now also J1.3 (B), J4.3 (B)
- net GND: now also J3.1 (A), J6.1 (A)
- net A12: now reaches U2.2 (A12)
- net A12: now also U1.2 (A12), U3.K (A12), J2.3 (B), J5.3 (B)
- net at U2.20 (~{CE}): now also J6.2 (C)
- net C1HIGH: now reaches U2.22 (~{OE})
- net C1HIGH: now also U3.6 (C1HIGH)
- net at U2.23 (A11): now also J5.2 (C)
- net at U2.26 (A13): now also J4.2 (C)
- net at U1.20 (~{CE}): now also J3.2 (C)
- net C1LOW: now reaches U1.22 (~{OE})
- net C1LOW: now also U3.B (/C1LOW)
- net at U1.23 (A11): now also J2.2 (C)
- net at U1.26 (A13): now also J1.2 (C)
- net A13: now reaches U3.J (A13)
- net A13: now also J1.1 (A), J4.1 (A)
- net A11: now reaches U3.L (A11)
- net A11: now also J2.1 (A), J3.3 (B), J5.1 (A), J6.3 (B)
- no-connect marks 3 -> 20
Other:
- moved on the sheet: U1, U2, U3

Commit message: Work in progress.
Parts:
- removed U4: 23128, symbol hackup:23128
- U1, U2: symbol Memory_EPROM:27C512 -> C264Cart:23128
Connections:
- net +5V: now also U1.27 (CS3*), U2.27 (CS3*)
- no-connect marks 20 -> 22
Other:
- company: (none) -> www.hackup.net
- title: (none) -> C264Cart - Artwork No. 310189 Replica
Changed lines of the file:
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@@
 (kicad_sch (version 20230121) (generator eeschema)
   (paper "A4")
+  (title_block
+    (title "C264Cart - Artwork No. 310189 Replica")
+    (rev "1")
+    (company "www.hackup.net")
+  )
   (junction (at 185.42 31.75) (diameter 0) (color 0 0 0 0)
   )
@@
   (no_connect (at 101.6 109.22))
   (no_connect (at 101.6 68.58))
+  (no_connect (at 218.44 88.9))
   (no_connect (at 63.5 63.5))
   (no_connect (at 63.5 60.96))
@@
   (no_connect (at 101.6 60.96))
   (no_connect (at 63.5 111.76))
+  (no_connect (at 158.75 88.9))
   (no_connect (at 101.6 63.5))
   (no_connect (at 101.6 58.42))
@@
     (stroke (width 0) (type default))
   )
+  (wire (pts (xy 214.63 93.98) (xy 218.44 93.98))
+    (stroke (width 0) (type default))
+  )
   (bus (pts (xy 212.09 73.66) (xy 212.09 76.2))
     (stroke (width 0) (type default))
@@
   )
   (bus (pts (xy 212.09 39.37) (xy 212.09 50.8))
+    (stroke (width 0) (type default))
+  )
+  (wire (pts (xy 154.94 93.98) (xy 158.75 93.98))
     (stroke (width 0) (type default))
   )
@@
     )
   )
+  (symbol (lib_id "power:+5V") (at 214.63 93.98 0) (mirror y) (unit 1)
+    (in_bom yes) (on_board yes) (dnp no) (fields_autoplaced)
+    (property "Reference" "#PWR014" (at 214.63 97.79 0)
+      (effects (font (size 1.27 1.27)) hide)
+    )
+    (property "Value" "+5V" (at 214.63 89.8469 0)
+      (effects (font (size 1.27 1.27)))
+    )
+    (property "Footprint" "" (at 214.63 93.98 0)
+      (effects (font (size 1.27 1.27)) hide)
+    )
+    (property "Datasheet" "" (at 214.63 93.98 0)
+      (effects (font (size 1.27 1.27)) hide)
+    )
+    (pin "1")
+    (instances
+      (project "C264Cart"
+        (path "/7006651b-1f52-4ff6-87a6-d875cc82c860"
+          (reference "#PWR014") (unit 1)
+        )
+      )
+    )
+  )
   (symbol (lib_id "power:+5V") (at 168.91 48.26 0) (unit 1)
     (in_bom yes) (on_board yes) (dnp no) (fields_autoplaced)
@@
     )
   )
-  (symbol (lib_id "Memory_EPROM:27C512") (at 228.6 76.2 0) (unit 1)
+  (symbol (lib_id "C264Cart:23128") (at 228.6 76.2 0) (unit 1)
     (in_bom yes) (on_board yes) (dnp no) (fields_autoplaced)
     (property "Reference" "U2" (at 230.7941 46.6557 0)
@@
     )
   )
-  (symbol (lib_id "hackup:23128") (at 17.78 171.45 0) (unit 1)
-    (in_bom yes) (on_board yes) (dnp no) (fields_autoplaced)
-    (property "Reference" "U4" (at 17.78 147.7698 0)
-      (effects (font (size 1.524 1.524)))
-    )
-    (property "Value" "23128" (at 17.78 150.6026 0)
-      (effects (font (size 1.524 1.524)))
-    )
-    (property "Footprint" "" (at 17.78 153.67 0)
-      (effects (font (size 1.524 1.524)) hide)
-    )
-    (property "Datasheet" "" (at 17.78 153.67 0)
-      (effects (font (size 1.524 1.524)) hide)
-    )
-    (pin "1")
-    (pin "15")
-    (pin "16")
-    (pin "17")
-    (pin "18")
-    (pin "19")
-    (pin "2")
-    (pin "20")
-    (pin "21")
-    (pin "22")
-    (pin "23")
-    (pin "24")
-    (pin "25")
-    (pin "26")
-    (pin "27")
-    (pin "28")
-    (pin "10")
-    (pin "11")
-    (pin "12")
-    (pin "13")
-    (pin "14")
-    (pin "3")
-    (pin "4")
-    (pin "5")
-    (pin "6")
-    (pin "7")
-    (pin "8")
-    (pin "9")
-    (instances
-      (project "C264Cart"
-        (path "/7006651b-1f52-4ff6-87a6-d875cc82c860"
-          (reference "U4") (unit 1)
-        )
-      )
-    )
-  )
   (symbol (lib_id "Jumper:SolderJumper_3_Bridged12") (at 212.09 119.38 0) (mirror x) (unit 1)
     (in_bom yes) (on_board yes) (dnp no)
@@
     )
   )
-  (symbol (lib_id "Memory_EPROM:27C512") (at 168.91 76.2 0) (unit 1)
+  (symbol (lib_id "C264Cart:23128") (at 168.91 76.2 0) (unit 1)
     (in_bom yes) (on_board yes) (dnp no) (fields_autoplaced)
     (property "Reference" "U1" (at 171.1041 46.6557 0)
@@
         )
       )
+    )
+  )
+  (symbol (lib_id "power:+5V") (at 154.94 93.98 0) (mirror y) (unit 1)
+    (in_bom yes) (on_board yes) (dnp no) (fields_autoplaced)
+    (property "Reference" "#PWR013" (at 154.94 97.79 0)
+      (effects (font (size 1.27 1.27)) hide)
+    )
+    (property "Value" "+5V" (at 154.94 89.8469 0)
+      (effects (font (size 1.27 1.27)))
+    )
+    (property "Footprint" "" (at 154.94 93.98 0)
+      (effects (font (size 1.27 1.27)) hide)
+    )
+    (property "Datasheet" "" (at 154.94 93.98 0)
+      (effects (font (size 1.27 1.27)) hide)
+    )
+    (pin "1")
+    (instances
+      (project "C264Cart"
+        (path "/7006651b-1f52-4ff6-87a6-d875cc82c860"
+          (reference "#PWR013") (unit 1)
+        )
+      )

Commit message: Work in progress.
Parts:
- added C1: 100n, Capacitor_THT:C_Disc_D6.0mm_W2.5mm_P5.00mm, symbol Device:C
Connections:
- net +5V: now also U1.1 (NC), U2.1 (NC), C1.1
- net GND: now also C1.2
- no-connect marks 22 -> 20
Changed lines of the file:
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@@
   (junction (at 152.4 39.37) (diameter 0) (color 0 0 0 0)
   )
+  (junction (at 217.17 93.98) (diameter 0) (color 0 0 0 0)
+  )
   (junction (at 134.62 133.35) (diameter 0) (color 0 0 0 0)
   )
   (junction (at 120.65 114.3) (diameter 0) (color 0 0 0 0)
+  )
+  (junction (at 157.48 93.98) (diameter 0) (color 0 0 0 0)
   )
   (junction (at 120.65 121.92) (diameter 0) (color 0 0 0 0)
@@
   (no_connect (at 101.6 109.22))
   (no_connect (at 101.6 68.58))
-  (no_connect (at 218.44 88.9))
   (no_connect (at 63.5 63.5))
   (no_connect (at 63.5 60.96))
@@
   (no_connect (at 101.6 60.96))
   (no_connect (at 63.5 111.76))
-  (no_connect (at 158.75 88.9))
   (no_connect (at 101.6 63.5))
   (no_connect (at 101.6 58.42))
@@
     (stroke (width 0) (type default))
   )
+  (wire (pts (xy 157.48 88.9) (xy 157.48 93.98))
+    (stroke (width 0) (type default))
+  )
   (wire (pts (xy 194.31 130.81) (xy 194.31 133.35))
     (stroke (width 0) (type default))
@@
     (stroke (width 0) (type default))
   )
+  (wire (pts (xy 158.75 88.9) (xy 157.48 88.9))
+    (stroke (width 0) (type default))
+  )
   (wire (pts (xy 120.65 114.3) (xy 120.65 121.92))
     (stroke (width 0) (type default))
@@
     (stroke (width 0) (type default))
   )
+  (wire (pts (xy 217.17 93.98) (xy 218.44 93.98))
+    (stroke (width 0) (type default))
+  )
   (bus (pts (xy 152.4 60.96) (xy 152.4 63.5))
     (stroke (width 0) (type default))
@@
     (stroke (width 0) (type default))
   )
+  (wire (pts (xy 157.48 93.98) (xy 158.75 93.98))
+    (stroke (width 0) (type default))
+  )
   (wire (pts (xy 179.07 66.04) (xy 182.88 66.04))
     (stroke (width 0) (type default))
   )
-  (wire (pts (xy 214.63 93.98) (xy 218.44 93.98))
+  (wire (pts (xy 214.63 93.98) (xy 217.17 93.98))
     (stroke (width 0) (type default))
   )
@@
     (stroke (width 0) (type default))
   )
-  (wire (pts (xy 154.94 93.98) (xy 158.75 93.98))
+  (wire (pts (xy 154.94 93.98) (xy 157.48 93.98))
     (stroke (width 0) (type default))
   )
@@
     (stroke (width 0) (type default))
   )
+  (wire (pts (xy 218.44 88.9) (xy 217.17 88.9))
+    (stroke (width 0) (type default))
+  )
   (wire (pts (xy 101.6 76.2) (xy 110.49 76.2))
     (stroke (width 0) (type default))
@@
   )
   (wire (pts (xy 156.21 99.06) (xy 158.75 99.06))
+    (stroke (width 0) (type default))
+  )
+  (wire (pts (xy 217.17 88.9) (xy 217.17 93.98))
     (stroke (width 0) (type default))
   )
@@
         (path "/7006651b-1f52-4ff6-87a6-d875cc82c860"
           (reference "#PWR07") (unit 1)
+        )
+      )
+    )
+  )
+  (symbol (lib_id "power:GND") (at 261.62 49.53 0) (unit 1)
+    (in_bom yes) (on_board yes) (dnp no) (fields_autoplaced)
+    (property "Reference" "#PWR016" (at 261.62 55.88 0)
+      (effects (font (size 1.27 1.27)) hide)
+    )
+    (property "Value" "GND" (at 261.62 53.6631 0)
+      (effects (font (size 1.27 1.27)))
+    )
+    (property "Footprint" "" (at 261.62 49.53 0)
+      (effects (font (size 1.27 1.27)) hide)
+    )
+    (property "Datasheet" "" (at 261.62 49.53 0)
+      (effects (font (size 1.27 1.27)) hide)
+    )
+    (pin "1")
+    (instances
+      (project "C264Cart"
+        (path "/7006651b-1f52-4ff6-87a6-d875cc82c860"
+          (reference "#PWR016") (unit 1)
         )
       )
@@
         )
       )
+    )
+  )
+  (symbol (lib_id "Device:C") (at 261.62 45.72 0) (unit 1)
+    (in_bom yes) (on_board yes) (dnp no) (fields_autoplaced)
+    (property "Reference" "C1" (at 264.541 44.5079 0)
+      (effects (font (size 1.27 1.27)) (justify left))
+    )
+    (property "Value" "100n" (at 264.541 46.9321 0)
+      (effects (font (size 1.27 1.27)) (justify left))
+    )
+    (property "Footprint" "Capacitor_THT:C_Disc_D6.0mm_W2.5mm_P5.00mm" (at 262.5852 49.53 0)
+      (effects (font (size 1.27 1.27)) hide)
+    )
+    (property "Datasheet" "~" (at 261.62 45.72 0)
+      (effects (font (size 1.27 1.27)) hide)
+    )
+    (pin "1")
+    (pin "2")
+    (instances
+      (project "C264Cart"
+        (path "/7006651b-1f52-4ff6-87a6-d875cc82c860"
+          (reference "C1") (unit 1)
+        )
+      )
+    )
+  )
+  (symbol (lib_id "power:+5V") (at 261.62 41.91 0) (unit 1)
+    (in_bom yes) (on_board yes) (dnp no) (fields_autoplaced)
+    (property "Reference" "#PWR015" (at 261.62 45.72 0)
+      (effects (font (size 1.27 1.27)) hide)
+    )
+    (property "Value" "+5V" (at 261.62 37.7769 0)
+      (effects (font (size 1.27 1.27)))
+    )
+    (property "Footprint" "" (at 261.62 41.91 0)
+      (effects (font (size 1.27 1.27)) hide)
+    )
+    (property "Datasheet" "" (at 261.62 41.91 0)
+      (effects (font (size 1.27 1.27)) hide)
+    )
+    (pin "1")
+    (instances
+      (project "C264Cart"
+        (path "/7006651b-1f52-4ff6-87a6-d875cc82c860"
+          (reference "#PWR015") (unit 1)
+        )
+      )

Commit message: Work in progress.
Parts:
- added C2: 100n, Capacitor_THT:C_Disc_D6.0mm_W2.5mm_P5.00mm, symbol Device:C
Connections:
- net +5V: now also C2.1
- net GND: now also C2.2
Changed lines of the file:
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@@
+    )
+  )
+  (symbol (lib_id "Device:C") (at 275.59 45.72 0) (unit 1)
+    (in_bom yes) (on_board yes) (dnp no) (fields_autoplaced)
+    (property "Reference" "C2" (at 278.511 44.5079 0)
+      (effects (font (size 1.27 1.27)) (justify left))
+    )
+    (property "Value" "100n" (at 278.511 46.9321 0)
+      (effects (font (size 1.27 1.27)) (justify left))
+    )
+    (property "Footprint" "Capacitor_THT:C_Disc_D6.0mm_W2.5mm_P5.00mm" (at 276.5552 49.53 0)
+      (effects (font (size 1.27 1.27)) hide)
+    )
+    (property "Datasheet" "~" (at 275.59 45.72 0)
+      (effects (font (size 1.27 1.27)) hide)
+    )
+    (pin "1")
+    (pin "2")
+    (instances
+      (project "C264Cart"
+        (path "/7006651b-1f52-4ff6-87a6-d875cc82c860"
+          (reference "C2") (unit 1)
+        )
+      )
     )
   )
@@
     )
   )
+  (symbol (lib_id "power:+5V") (at 275.59 41.91 0) (unit 1)
+    (in_bom yes) (on_board yes) (dnp no) (fields_autoplaced)
+    (property "Reference" "#PWR017" (at 275.59 45.72 0)
+      (effects (font (size 1.27 1.27)) hide)
+    )
+    (property "Value" "+5V" (at 275.59 37.7769 0)
+      (effects (font (size 1.27 1.27)))
+    )
+    (property "Footprint" "" (at 275.59 41.91 0)
+      (effects (font (size 1.27 1.27)) hide)
+    )
+    (property "Datasheet" "" (at 275.59 41.91 0)
+      (effects (font (size 1.27 1.27)) hide)
+    )
+    (pin "1")
+    (instances
+      (project "C264Cart"
+        (path "/7006651b-1f52-4ff6-87a6-d875cc82c860"
+          (reference "#PWR017") (unit 1)
+        )
+      )
+    )
+  )
   (symbol (lib_id "power:PWR_FLAG") (at 261.62 24.13 180) (unit 1)
     (in_bom yes) (on_board yes) (dnp no) (fields_autoplaced)
@@
         )
       )
+    )
+  )
+  (symbol (lib_id "power:GND") (at 275.59 49.53 0) (unit 1)
+    (in_bom yes) (on_board yes) (dnp no) (fields_autoplaced)
+    (property "Reference" "#PWR018" (at 275.59 55.88 0)
+      (effects (font (size 1.27 1.27)) hide)
+    )
+    (property "Value" "GND" (at 275.59 53.6631 0)
+      (effects (font (size 1.27 1.27)))
+    )
+    (property "Footprint" "" (at 275.59 49.53 0)
+      (effects (font (size 1.27 1.27)) hide)
+    )
+    (property "Datasheet" "" (at 275.59 49.53 0)
+      (effects (font (size 1.27 1.27)) hide)
+    )
+    (pin "1")
+    (instances
+      (project "C264Cart"
+        (path "/7006651b-1f52-4ff6-87a6-d875cc82c860"
+          (reference "#PWR018") (unit 1)
+        )
+      )

Commit message: Clean up schematics.
Parts:
- U1, U2: value 27C512 -> 23128
Other:
- moved on the sheet: J1, J2, J3, U1, U2, U3
