File: C264Cart.kicad_pcb (KiCad board)
At the start: 2 copper layers, 55.8 x 64.7 mm, 14 parts, among them U1 27C040, U3 264-Exp-Port

Commit message: JLC order number location.
Other:
- board text added: "JLCJLCJLCJLC"

Commit message: Minor layout fixes.
Routing:
- net /CE: vias 1 -> 0
Changed lines of the file:
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@@
   (gr_arc (start 135.661401 80.120458) (mid 135.255448 78.9178) (end 135.586532 77.692416)
     (stroke (width 0.15) (type default)) (layer "F.SilkS"))
-  (gr_line (start 102.0594 44.4018) (end 157.8594 44.4018)
-    (stroke (width 0.15) (type default)) (layer "Dwgs.User"))
   (gr_arc (start 157.8594 124.8018) (mid 157.683664 125.226064) (end 157.2594 125.4018)
     (stroke (width 0.1) (type default)) (layer "Edge.Cuts"))
@@
   (segment (start 102.7594 98.22046) (end 102.7594 90.60046) (width 1) (layer "B.Cu") (net 12))
   (segment (start 148.6154 74.8538) (end 151.1554 74.8538) (width 1) (layer "B.Cu") (net 12))
-  (segment (start 142.621 74.8792) (end 142.5956 74.8538) (width 0.25) (layer "B.Cu") (net 12))
   (segment (start 154.4444 87.3122) (end 154.4444 83.7568) (width 0.25) (layer "B.Cu") (net 12))
   (segment (start 155.2194 88.0872) (end 154.4444 87.3122) (width 0.25) (layer "B.Cu") (net 12))
@@
   (segment (start 123.409391 92.7608) (end 138.6964 92.7608) (width 0.25) (layer "F.Cu") (net 54))
   (segment (start 137.4394 80.4418) (end 138.6144 81.6168) (width 0.25) (layer "F.Cu") (net 54))
-  (via (at 138.6964 92.7608) (size 0.8) (drill 0.4) (layers "F.Cu" "B.Cu") (net 54))
   (segment (start 106.9594 90.6018) (end 108.0844 91.7268) (width 0.25) (layer "B.Cu") (net 54))
   (segment (start 108.0844 94.5568) (end 106.9594 95.6818) (width 0.25) (layer "B.Cu") (net 54))
